File: cad/dlr_carrier-charger.kicad_sch (KiCad schematic)
At the start: 25 parts, among them J1 PV_IN, Q1 DMN4035L-7, Q2 DMN4035L-7, U8 BQ24650RVAR

Commit message: 🩺 fix(schematic): match hierarchical label type to the sheet pin
The 117 KiCad 9 errors were a type mismatch, not the hierarchy metadata: every
child hierarchical label was written as `(shape input)` while the root's sheet pins
are bidirectional. KiCad's hier_label_mismatch check compares electrical type as
well as name, so on KiCad 9 every cross-sheet net failed, and the root labels then
read as dangling. KiCad 10 tolerates the mismatch, which is why it passed here.

kicad-sch-api 0.5.6 accepts a shape argument on add_hierarchical_label and ignores
it — the third serialization bug worked around in this generator — so the shape is
rewritten in the saved sheet.

Co-Authored-By: Claude Opus 5 <noreply@anthropic.com>
Claude-Session: https://claude.ai/code/session_011xr7VCL7rkJj2WE2uQF7sF
Changed lines of the file:
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@@
 		(instances
 			(project "SOLAR MPPT CHARGER"
-				(path "/1973253c-82cd-4127-8fdc-bf7042356fee"
+				(path "/40c61e59-64f7-482c-bac7-2bc5cddc1686"
 					(reference "C1")
 					(unit 1)
@@
 		(instances
 			(project "SOLAR MPPT CHARGER"
-				(path "/1973253c-82cd-4127-8fdc-bf7042356fee"
+				(path "/40c61e59-64f7-482c-bac7-2bc5cddc1686"
 					(reference "C2")
 					(unit 1)
@@
 		(instances
 			(project "SOLAR MPPT CHARGER"
-				(path "/1973253c-82cd-4127-8fdc-bf7042356fee"
+				(path "/40c61e59-64f7-482c-bac7-2bc5cddc1686"
 					(reference "C3")
 					(unit 1)
@@
 		(instances
 			(project "SOLAR MPPT CHARGER"
-				(path "/1973253c-82cd-4127-8fdc-bf7042356fee"
+				(path "/40c61e59-64f7-482c-bac7-2bc5cddc1686"
 					(reference "C31")
 					(unit 1)
@@
 		(instances
 			(project "SOLAR MPPT CHARGER"
-				(path "/1973253c-82cd-4127-8fdc-bf7042356fee"
+				(path "/40c61e59-64f7-482c-bac7-2bc5cddc1686"
 					(reference "C32")
 					(unit 1)
@@
 		(instances
 			(project "SOLAR MPPT CHARGER"
-				(path "/1973253c-82cd-4127-8fdc-bf7042356fee"
+				(path "/40c61e59-64f7-482c-bac7-2bc5cddc1686"
 					(reference "C33")
 					(unit 1)
@@
 		(instances
 			(project "SOLAR MPPT CHARGER"
-				(path "/1973253c-82cd-4127-8fdc-bf7042356fee"
+				(path "/40c61e59-64f7-482c-bac7-2bc5cddc1686"
 					(reference "C34")
 					(unit 1)
@@
 		(instances
 			(project "SOLAR MPPT CHARGER"
-				(path "/1973253c-82cd-4127-8fdc-bf7042356fee"
+				(path "/40c61e59-64f7-482c-bac7-2bc5cddc1686"
 					(reference "C35")
 					(unit 1)
@@
 		(instances
 			(project "SOLAR MPPT CHARGER"
-				(path "/1973253c-82cd-4127-8fdc-bf7042356fee"
+				(path "/40c61e59-64f7-482c-bac7-2bc5cddc1686"
 					(reference "D1")
 					(unit 1)
@@
 		(instances
 			(project "SOLAR MPPT CHARGER"
-				(path "/1973253c-82cd-4127-8fdc-bf7042356fee"
+				(path "/40c61e59-64f7-482c-bac7-2bc5cddc1686"
 					(reference "D4")
 					(unit 1)
@@
 		(instances
 			(project "SOLAR MPPT CHARGER"
-				(path "/1973253c-82cd-4127-8fdc-bf7042356fee"
+				(path "/40c61e59-64f7-482c-bac7-2bc5cddc1686"
 					(reference "J1")
 					(unit 1)
@@
 		(instances
 			(project "SOLAR MPPT CHARGER"
-				(path "/1973253c-82cd-4127-8fdc-bf7042356fee"
+				(path "/40c61e59-64f7-482c-bac7-2bc5cddc1686"
 					(reference "L1")
 					(unit 1)
@@
 		(instances
 			(project "SOLAR MPPT CHARGER"
-				(path "/1973253c-82cd-4127-8fdc-bf7042356fee"
+				(path "/40c61e59-64f7-482c-bac7-2bc5cddc1686"
 					(reference "Q1")
 					(unit 1)
@@
 		(instances
 			(project "SOLAR MPPT CHARGER"
-				(path "/1973253c-82cd-4127-8fdc-bf7042356fee"
+				(path "/40c61e59-64f7-482c-bac7-2bc5cddc1686"
 					(reference "Q2")
 					(unit 1)
@@
 		(instances
 			(project "SOLAR MPPT CHARGER"
-				(path "/1973253c-82cd-4127-8fdc-bf7042356fee"
+				(path "/40c61e59-64f7-482c-bac7-2bc5cddc1686"
 					(reference "R1")
 					(unit 1)
@@
 		(instances
 			(project "SOLAR MPPT CHARGER"
-				(path "/1973253c-82cd-4127-8fdc-bf7042356fee"
+				(path "/40c61e59-64f7-482c-bac7-2bc5cddc1686"
 					(reference "R17")
 					(unit 1)
@@
 		(instances
 			(project "SOLAR MPPT CHARGER"
-				(path "/1973253c-82cd-4127-8fdc-bf7042356fee"
+				(path "/40c61e59-64f7-482c-bac7-2bc5cddc1686"
 					(reference "R18")
 					(unit 1)
@@
 		(instances
 			(project "SOLAR MPPT CHARGER"
-				(path "/1973253c-82cd-4127-8fdc-bf7042356fee"
+				(path "/40c61e59-64f7-482c-bac7-2bc5cddc1686"
 					(reference "R19")
 					(unit 1)
@@
 		(instances
 			(project "SOLAR MPPT CHARGER"
-				(path "/1973253c-82cd-4127-8fdc-bf7042356fee"
+				(path "/40c61e59-64f7-482c-bac7-2bc5cddc1686"
 					(reference "R20")
 					(unit 1)
@@
 		(instances
 			(project "SOLAR MPPT CHARGER"
-				(path "/1973253c-82cd-4127-8fdc-bf7042356fee"
+				(path "/40c61e59-64f7-482c-bac7-2bc5cddc1686"
 					(reference "R21")
 					(unit 1)
@@
 		(instances
 			(project "SOLAR MPPT CHARGER"
-				(path "/1973253c-82cd-4127-8fdc-bf7042356fee"
+				(path "/40c61e59-64f7-482c-bac7-2bc5cddc1686"
 					(reference "R22")
 					(unit 1)
@@
 		(instances
 			(project "SOLAR MPPT CHARGER"
-				(path "/1973253c-82cd-4127-8fdc-bf7042356fee"
+				(path "/40c61e59-64f7-482c-bac7-2bc5cddc1686"
 					(reference "R23")
 					(unit 1)
@@
 		(instances
 			(project "SOLAR MPPT CHARGER"
-				(path "/1973253c-82cd-4127-8fdc-bf7042356fee"
+				(path "/40c61e59-64f7-482c-bac7-2bc5cddc1686"
 					(reference "R24")
 					(unit 1)
@@
 		(instances
 			(project "SOLAR MPPT CHARGER"
-				(path "/1973253c-82cd-4127-8fdc-bf7042356fee"
+				(path "/40c61e59-64f7-482c-bac7-2bc5cddc1686"
 					(reference "R25")
 					(unit 1)
@@
 		(instances
 			(project "SOLAR MPPT CHARGER"
-				(path "/1973253c-82cd-4127-8fdc-bf7042356fee"
+				(path "/40c61e59-64f7-482c-bac7-2bc5cddc1686"
 					(reference "U8")
 					(unit 1)
@@
 		(instances
 			(project "SOLAR MPPT CHARGER"
-				(path "/1973253c-82cd-4127-8fdc-bf7042356fee"
+				(path "/40c61e59-64f7-482c-bac7-2bc5cddc1686"
 					(reference "#PWR001")
 					(unit 1)
@@
 		(instances
 			(project "SOLAR MPPT CHARGER"
-				(path "/1973253c-82cd-4127-8fdc-bf7042356fee"
+				(path "/40c61e59-64f7-482c-bac7-2bc5cddc1686"
 					(reference "#PWR002")
 					(unit 1)
@@
 		(instances
 			(project "SOLAR MPPT CHARGER"
-				(path "/1973253c-82cd-4127-8fdc-bf7042356fee"
+				(path "/40c61e59-64f7-482c-bac7-2bc5cddc1686"
 					(reference "#FLG001")
 					(unit 1)
@@
 		(instances
 			(project "SOLAR MPPT CHARGER"
-				(path "/1973253c-82cd-4127-8fdc-bf7042356fee"
+				(path "/40c61e59-64f7-482c-bac7-2bc5cddc1686"
 					(reference "#PWR003")
 					(unit 1)
@@
 		(instances
 			(project "SOLAR MPPT CHARGER"
-				(path "/1973253c-82cd-4127-8fdc-bf7042356fee"
+				(path "/40c61e59-64f7-482c-bac7-2bc5cddc1686"
 					(reference "#PWR004")
 					(unit 1)
@@
 		(instances
 			(project "SOLAR MPPT CHARGER"
-				(path "/1973253c-82cd-4127-8fdc-bf7042356fee"
+				(path "/40c61e59-64f7-482c-bac7-2bc5cddc1686"
 					(reference "#PWR005")
 					(unit 1)
@@
 		(instances
 			(project "SOLAR MPPT CHARGER"
-				(path "/1973253c-82cd-4127-8fdc-bf7042356fee"
+				(path "/40c61e59-64f7-482c-bac7-2bc5cddc1686"
 					(reference "#PWR006")
 					(unit 1)
@@
 		(instances
 			(project "SOLAR MPPT CHARGER"
-				(path "/1973253c-82cd-4127-8fdc-bf7042356fee"
+				(path "/40c61e59-64f7-482c-bac7-2bc5cddc1686"
 					(reference "#PWR007")
 					(unit 1)
@@
 		(instances
 			(project "SOLAR MPPT CHARGER"
-				(path "/1973253c-82cd-4127-8fdc-bf7042356fee"
+				(path "/40c61e59-64f7-482c-bac7-2bc5cddc1686"
 					(reference "#PWR008")
 					(unit 1)
@@
 		(instances
 			(project "SOLAR MPPT CHARGER"
-				(path "/1973253c-82cd-4127-8fdc-bf7042356fee"
+				(path "/40c61e59-64f7-482c-bac7-2bc5cddc1686"
 					(reference "#PWR009")
 					(unit 1)
@@
 		(instances
 			(project "SOLAR MPPT CHARGER"
-				(path "/1973253c-82cd-4127-8fdc-bf7042356fee"
+				(path "/40c61e59-64f7-482c-bac7-2bc5cddc1686"
 					(reference "#PWR010")
 					(unit 1)
@@
 		(instances
 			(project "SOLAR MPPT CHARGER"
-				(path "/1973253c-82cd-4127-8fdc-bf7042356fee"
+				(path "/40c61e59-64f7-482c-bac7-2bc5cddc1686"
 					(reference "#PWR011")
 					(unit 1)
@@
 		(instances
 			(project "SOLAR MPPT CHARGER"
-				(path "/1973253c-82cd-4127-8fdc-bf7042356fee"
+				(path "/40c61e59-64f7-482c-bac7-2bc5cddc1686"
 					(reference "#PWR012")
 					(unit 1)
@@
 		(instances
 			(project "SOLAR MPPT CHARGER"
-				(path "/1973253c-82cd-4127-8fdc-bf7042356fee"
+				(path "/40c61e59-64f7-482c-bac7-2bc5cddc1686"
 					(reference "#PWR013")
 					(unit 1)
@@
 		(instances
 			(project "SOLAR MPPT CHARGER"
-				(path "/1973253c-82cd-4127-8fdc-bf7042356fee"
+				(path "/40c61e59-64f7-482c-bac7-2bc5cddc1686"
 					(reference "#PWR014")
 					(unit 1)
@@
 		(instances
 			(project "SOLAR MPPT CHARGER"
-				(path "/1973253c-82cd-4127-8fdc-bf7042356fee"
+				(path "/40c61e59-64f7-482c-bac7-2bc5cddc1686"
 					(reference "#PWR015")
 					(unit 1)
@@
 		(instances
 			(project "SOLAR MPPT CHARGER"
-				(path "/1973253c-82cd-4127-8fdc-bf7042356fee"
+				(path "/40c61e59-64f7-482c-bac7-2bc5cddc1686"
 					(reference "#FLG002")
 					(unit 1)
@@
 	)
 	(hierarchical_label "CHG_STAT1"
-		(shape input)
+		(shape bidirectional)
 		(at 114.3 274.32 270)
 		(effects
@@
 	)
 	(hierarchical_label "CHG_STAT1"
-		(shape input)
+		(shape bidirectional)
 		(at 238.76 275.59 0)
 		(effects
@@
 	)
 	(hierarchical_label "CHG_STAT2"
-		(shape input)
+		(shape bidirectional)
 		(at 165.1 274.32 270)
 		(effects
@@
 	)
 	(hierarchical_label "CHG_STAT2"
-		(shape input)
+		(shape bidirectional)
 		(at 238.76 278.13 0)
 		(effects
@@
 	)
 	(hierarchical_label "VBAT"
-		(shape input)
+		(shape bidirectional)
 		(at 165.1 60.96 90)
 		(effects
@@
 	)
 	(hierarchical_label "VBAT"
-		(shape input)
+		(shape bidirectional)
 		(at 368.3 83.82 270)
 		(effects
@@
 	)
 	(hierarchical_label "VBAT"
-		(shape input)
+		(shape bidirectional)
 		(at 63.5 124.46 90)
 		(effects
@@
 	)
 	(hierarchical_label "VBAT"
-		(shape input)
+		(shape bidirectional)
 		(at 63.5 210.82 270)
 		(effects
@@
 	)
 	(hierarchical_label "VBAT"
-		(shape input)
+		(shape bidirectional)
 		(at 266.7 187.96 90)
 		(effects
@@
 	)
 	(hierarchical_label "VBAT"
-		(shape input)
+		(shape bidirectional)
 		(at 238.76 262.89 0)
 		(effects
@@
 	)
 	(sheet_instances
-		(path "/5d35d880-5624-4087-ac0f-9ed923009ccf"
+		(path "/ff7de960-6bdd-4734-b765-9a85f5be0719"
 			(page "2")
 		)
