File: cad/dlr_carrier-som.kicad_sch (KiCad schematic)
At the start: 5 parts, among them J5 CM4_J2

Commit message: 🩺 refactor(schematic): cross-sheet nets via global labels, no sheet pins
Three attempts at making the hierarchical sheet-pin mechanism pass KiCad 9 failed
(project name, instance paths, label type), so the mechanism goes. Cross-sheet nets
now connect by name through global labels on the child sheets; the root carries
sheet symbols only — no pins, no stub wires, no labels.

That removes the whole hier_label_mismatch / label_dangling class rather than
chasing it, and it matches the connectivity style the generate-schematic skill
already prescribes for this project ("all inter-block connections use net labels").

kicad-sch-api's add_global_label still does not serialize, so the labels are emitted
as hierarchical and rewritten in the saved sheet.

Co-Authored-By: Claude Opus 5 <noreply@anthropic.com>
Claude-Session: https://claude.ai/code/session_011xr7VCL7rkJj2WE2uQF7sF
Changed lines of the file:
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@@
 		(instances
 			(project "CM4 SoM"
-				(path "/8bad8029-d445-45ba-bfa9-ecca933e2f0a"
+				(path "/7d682eb5-d59b-45bd-8ff7-9e2b95ee6b69"
 					(reference "J5")
 					(unit 1)
@@
 		(instances
 			(project "CM4 SoM"
-				(path "/8bad8029-d445-45ba-bfa9-ecca933e2f0a"
+				(path "/7d682eb5-d59b-45bd-8ff7-9e2b95ee6b69"
 					(reference "C14")
 					(unit 1)
@@
 		(instances
 			(project "CM4 SoM"
-				(path "/8bad8029-d445-45ba-bfa9-ecca933e2f0a"
+				(path "/7d682eb5-d59b-45bd-8ff7-9e2b95ee6b69"
 					(reference "C15")
 					(unit 1)
@@
 		(instances
 			(project "CM4 SoM"
-				(path "/8bad8029-d445-45ba-bfa9-ecca933e2f0a"
+				(path "/7d682eb5-d59b-45bd-8ff7-9e2b95ee6b69"
 					(reference "C16")
 					(unit 1)
@@
 		(instances
 			(project "CM4 SoM"
-				(path "/8bad8029-d445-45ba-bfa9-ecca933e2f0a"
+				(path "/7d682eb5-d59b-45bd-8ff7-9e2b95ee6b69"
 					(reference "C17")
 					(unit 1)
@@
 		(instances
 			(project "CM4 SoM"
-				(path "/8bad8029-d445-45ba-bfa9-ecca933e2f0a"
+				(path "/7d682eb5-d59b-45bd-8ff7-9e2b95ee6b69"
 					(reference "#PWR001")
 					(unit 1)
@@
 		(instances
 			(project "CM4 SoM"
-				(path "/8bad8029-d445-45ba-bfa9-ecca933e2f0a"
+				(path "/7d682eb5-d59b-45bd-8ff7-9e2b95ee6b69"
 					(reference "#PWR002")
 					(unit 1)
@@
 		(instances
 			(project "CM4 SoM"
-				(path "/8bad8029-d445-45ba-bfa9-ecca933e2f0a"
+				(path "/7d682eb5-d59b-45bd-8ff7-9e2b95ee6b69"
 					(reference "#PWR003")
 					(unit 1)
@@
 		(instances
 			(project "CM4 SoM"
-				(path "/8bad8029-d445-45ba-bfa9-ecca933e2f0a"
+				(path "/7d682eb5-d59b-45bd-8ff7-9e2b95ee6b69"
 					(reference "#PWR004")
 					(unit 1)
@@
 		(instances
 			(project "CM4 SoM"
-				(path "/8bad8029-d445-45ba-bfa9-ecca933e2f0a"
+				(path "/7d682eb5-d59b-45bd-8ff7-9e2b95ee6b69"
 					(reference "#PWR005")
 					(unit 1)
@@
 		(instances
 			(project "CM4 SoM"
-				(path "/8bad8029-d445-45ba-bfa9-ecca933e2f0a"
+				(path "/7d682eb5-d59b-45bd-8ff7-9e2b95ee6b69"
 					(reference "#PWR006")
 					(unit 1)
@@
 		(instances
 			(project "CM4 SoM"
-				(path "/8bad8029-d445-45ba-bfa9-ecca933e2f0a"
+				(path "/7d682eb5-d59b-45bd-8ff7-9e2b95ee6b69"
 					(reference "#PWR007")
 					(unit 1)
@@
 		(instances
 			(project "CM4 SoM"
-				(path "/8bad8029-d445-45ba-bfa9-ecca933e2f0a"
+				(path "/7d682eb5-d59b-45bd-8ff7-9e2b95ee6b69"
 					(reference "#PWR008")
 					(unit 1)
@@
 		(instances
 			(project "CM4 SoM"
-				(path "/8bad8029-d445-45ba-bfa9-ecca933e2f0a"
+				(path "/7d682eb5-d59b-45bd-8ff7-9e2b95ee6b69"
 					(reference "#PWR009")
 					(unit 1)
@@
 		(instances
 			(project "CM4 SoM"
-				(path "/8bad8029-d445-45ba-bfa9-ecca933e2f0a"
+				(path "/7d682eb5-d59b-45bd-8ff7-9e2b95ee6b69"
 					(reference "#PWR010")
 					(unit 1)
@@
 		(instances
 			(project "CM4 SoM"
-				(path "/8bad8029-d445-45ba-bfa9-ecca933e2f0a"
+				(path "/7d682eb5-d59b-45bd-8ff7-9e2b95ee6b69"
 					(reference "#PWR011")
 					(unit 1)
@@
 		(instances
 			(project "CM4 SoM"
-				(path "/8bad8029-d445-45ba-bfa9-ecca933e2f0a"
+				(path "/7d682eb5-d59b-45bd-8ff7-9e2b95ee6b69"
 					(reference "#PWR012")
 					(unit 1)
@@
 		(instances
 			(project "CM4 SoM"
-				(path "/8bad8029-d445-45ba-bfa9-ecca933e2f0a"
+				(path "/7d682eb5-d59b-45bd-8ff7-9e2b95ee6b69"
 					(reference "#PWR013")
 					(unit 1)
@@
 		(instances
 			(project "CM4 SoM"
-				(path "/8bad8029-d445-45ba-bfa9-ecca933e2f0a"
+				(path "/7d682eb5-d59b-45bd-8ff7-9e2b95ee6b69"
 					(reference "#PWR014")
 					(unit 1)
@@
 		(instances
 			(project "CM4 SoM"
-				(path "/8bad8029-d445-45ba-bfa9-ecca933e2f0a"
+				(path "/7d682eb5-d59b-45bd-8ff7-9e2b95ee6b69"
 					(reference "#PWR015")
 					(unit 1)
@@
 		(instances
 			(project "CM4 SoM"
-				(path "/8bad8029-d445-45ba-bfa9-ecca933e2f0a"
+				(path "/7d682eb5-d59b-45bd-8ff7-9e2b95ee6b69"
 					(reference "#PWR016")
 					(unit 1)
@@
 		(instances
 			(project "CM4 SoM"
-				(path "/8bad8029-d445-45ba-bfa9-ecca933e2f0a"
+				(path "/7d682eb5-d59b-45bd-8ff7-9e2b95ee6b69"
 					(reference "#PWR017")
 					(unit 1)
@@
 		(instances
 			(project "CM4 SoM"
-				(path "/8bad8029-d445-45ba-bfa9-ecca933e2f0a"
+				(path "/7d682eb5-d59b-45bd-8ff7-9e2b95ee6b69"
 					(reference "#PWR018")
 					(unit 1)
@@
 		(instances
 			(project "CM4 SoM"
-				(path "/8bad8029-d445-45ba-bfa9-ecca933e2f0a"
+				(path "/7d682eb5-d59b-45bd-8ff7-9e2b95ee6b69"
 					(reference "#PWR019")
 					(unit 1)
@@
 		(instances
 			(project "CM4 SoM"
-				(path "/8bad8029-d445-45ba-bfa9-ecca933e2f0a"
+				(path "/7d682eb5-d59b-45bd-8ff7-9e2b95ee6b69"
 					(reference "#PWR020")
 					(unit 1)
@@
 		)
 	)
-	(hierarchical_label "ANEMO_DE"
+	(global_label "ANEMO_DE"
 		(shape bidirectional)
 		(at 97.79 180.34 180)
@@
 		)
 	)
-	(hierarchical_label "ANEMO_UART_RX"
+	(global_label "ANEMO_UART_RX"
 		(shape bidirectional)
 		(at 125.73 175.26 0)
@@
 		)
 	)
-	(hierarchical_label "ANEMO_UART_TX"
+	(global_label "ANEMO_UART_TX"
 		(shape bidirectional)
 		(at 97.79 175.26 180)
@@
 		)
 	)
-	(hierarchical_label "CELL_EN"
+	(global_label "CELL_EN"
 		(shape bidirectional)
 		(at 97.79 154.94 180)
@@
 		)
 	)
-	(hierarchical_label "CELL_NET_STATUS"
+	(global_label "CELL_NET_STATUS"
 		(shape bidirectional)
 		(at 97.79 157.48 180)
@@
 		)
 	)
-	(hierarchical_label "CELL_PWRKEY"
+	(global_label "CELL_PWRKEY"
 		(shape bidirectional)
 		(at 97.79 160.02 180)
@@
 		)
 	)
-	(hierarchical_label "CELL_RESET"
+	(global_label "CELL_RESET"
 		(shape bidirectional)
 		(at 125.73 160.02 0)
@@
 		)
 	)
-	(hierarchical_label "CELL_STATUS"
+	(global_label "CELL_STATUS"
 		(shape bidirectional)
 		(at 125.73 162.56 0)
@@
 		)
 	)
-	(hierarchical_label "CHG_STAT1"
+	(global_label "CHG_STAT1"
 		(shape bidirectional)
 		(at 125.73 154.94 0)
@@
 		)
 	)
-	(hierarchical_label "CHG_STAT2"
+	(global_label "CHG_STAT2"
 		(shape bidirectional)
 		(at 125.73 172.72 0)
@@
 		)
 	)
-	(hierarchical_label "DBG_RX"
+	(global_label "DBG_RX"
 		(shape bidirectional)
 		(at 97.79 182.88 180)
@@
 		)
 	)
-	(hierarchical_label "DBG_TX"
+	(global_label "DBG_TX"
 		(shape bidirectional)
 		(at 125.73 180.34 0)
@@
 		)
 	)
-	(hierarchical_label "GPIO25_VSYNC"
+	(global_label "GPIO25_VSYNC"
 		(shape bidirectional)
 		(at 125.73 167.64 0)
@@
 		)
 	)
-	(hierarchical_label "GPIO4_DHT22"
+	(global_label "GPIO4_DHT22"
 		(shape bidirectional)
 		(at 97.79 149.86 180)
@@
 		)
 	)
-	(hierarchical_label "SCL1"
+	(global_label "SCL1"
 		(shape bidirectional)
 		(at 97.79 147.32 180)
@@
 		)
 	)
-	(hierarchical_label "SDA1"
+	(global_label "SDA1"
 		(shape bidirectional)
 		(at 97.79 144.78 180)
@@
 		)
 	)
-	(hierarchical_label "SHIFTER_OE"
+	(global_label "SHIFTER_OE"
 		(shape bidirectional)
 		(at 97.79 177.8 180)
@@
 		)
 	)
-	(hierarchical_label "SPI0_CE0"
+	(global_label "SPI0_CE0"
 		(shape bidirectional)
 		(at 125.73 170.18 0)
@@
 		)
 	)
-	(hierarchical_label "SPI0_MISO"
+	(global_label "SPI0_MISO"
 		(shape bidirectional)
 		(at 97.79 167.64 180)
@@
 		)
 	)
-	(hierarchical_label "SPI0_MOSI"
+	(global_label "SPI0_MOSI"
 		(shape bidirectional)
 		(at 97.79 165.1 180)
@@
 		)
 	)
-	(hierarchical_label "SPI0_SCLK"
+	(global_label "SPI0_SCLK"
 		(shape bidirectional)
 		(at 97.79 170.18 180)
@@
 		)
 	)
-	(hierarchical_label "UART_RX_3V3"
+	(global_label "UART_RX_3V3"
 		(shape bidirectional)
 		(at 125.73 152.4 0)
@@
 		)
 	)
-	(hierarchical_label "UART_TX_3V3"
+	(global_label "UART_TX_3V3"
 		(shape bidirectional)
 		(at 125.73 149.86 0)
@@
 		)
 	)
-	(hierarchical_label "USB_CMSN_DM"
+	(global_label "USB_CMSN_DM"
 		(shape bidirectional)
 		(at 97.79 187.96 180)
@@
 		)
 	)
-	(hierarchical_label "USB_CMSN_DP"
+	(global_label "USB_CMSN_DP"
 		(shape bidirectional)
 		(at 125.73 185.42 0)
@@
 		)
 	)
-	(hierarchical_label "USB_DM"
+	(global_label "USB_DM"
 		(shape bidirectional)
 		(at 125.73 190.5 0)
@@
 		)
 	)
-	(hierarchical_label "USB_DP"
+	(global_label "USB_DP"
 		(shape bidirectional)
 		(at 125.73 187.96 0)
@@
 	)
 	(sheet_instances
-		(path "/4a3e06bc-d7fd-4803-a708-54e05d93e811"
+		(path "/9a9446e4-a86f-49a2-bdd6-63e557d71cc1"
 			(page "4")
 		)
